File: esp32-c6-pico.kicad_sch (KiCad schematic)
At the start: 35 parts, among them U1 ESP32-C6, U3 W25Q32JVZPIQ, Y1 40MHz / CL=8pF

Commit message: Refine ESP32-C6 Pico layout and project handoff
Update the 20.5 x 32 mm layout, antenna and crystal placement, USB routing, via clearances, and silkscreen logos. Keep RF passives at 0201 and use 0402 for all other resistors and capacitors. Draw ESP32-C6 peripherals directly from U1 pins.

Refresh BOM, placement files, previews, validation reports, and project guidance. Exclude KiCad backup folders, autosaves, and local state on Windows and Linux.

Validation: ERC, DRC, and unconnected counts are zero; all 45 QA checks passed. Verify final file hashes and backup exclusions before commit.
Parts:
- added C21, C25: 1uF, Capacitor_SMD:C_0402_1005Metric, symbol Pico_Design:Device__C_Small
- added C26: 100nF, Capacitor_SMD:C_0402_1005Metric, symbol Pico_Design:Device__C_Small
- added C27, C28: DNP, Capacitor_SMD:C_0402_1005Metric, symbol Pico_Design:Device__C_Small
- added D2: WS2812B-2020, Pico:WS2812B_2020_Compact, symbol Pico_Design:LED__WS2812B-2020
- added R12, R13: 22R, Resistor_SMD:R_0402_1005Metric, symbol Pico_Design:Device__R_Small
- added R14: 499R, Resistor_SMD:R_0402_1005Metric, symbol Pico_Design:Device__R_Small
- added R15: 330R, Resistor_SMD:R_0402_1005Metric, symbol Pico_Design:Device__R_Small
- added R16: 100k, Resistor_SMD:R_0402_1005Metric, symbol Pico_Design:Device__R_Small
- added R7, R8, R9: 10k, Resistor_SMD:R_0402_1005Metric, symbol Pico_Design:Device__R_Small
- added SW1: RESET, Button_Switch_SMD:SW_Push_1P1T_NO_CK_KMR2, symbol Pico_Design:Switch__SW_Push
- added SW2: BOOT, Button_Switch_SMD:SW_Push_1P1T_NO_CK_KMR2, symbol Pico_Design:Switch__SW_Push
- added U4: SN74LV1T125, Package_TO_SOT_SMD:SOT-23-5, symbol Pico_Design:Pico_Custom__SN74LV1T125
- AE1: AssemblyNote Pad 2 has open tuning copper, never connect to ground; 18x9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 -> Pad 2 stays open with axial end copper; horizontal prototyp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
- C19: footprint Capacitor_SMD:C_0603_1608Metric -> Capacitor_SMD:C_0402_1005Metric; AssemblyNote U1 pin 2 local bulk -> U1 pin 2 local bulk; 0402, 10 V minimum; verify effective c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
- C20: footprint Capacitor_SMD:C_0603_1608Metric -> Capacitor_SMD:C_0402_1005Metric; AssemblyNote U1 pin 3 local bulk -> U1 pin 3 local bulk; 0402, 10 V minimum; verify effective c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
- C8: footprint Capacitor_SMD:C_0603_1608Metric -> Capacitor_SMD:C_0402_1005Metric; AssemblyNote Main bulk; X7R 10 V minimum -> Main bulk; 0402, 10 V minimum; X5R reference; verify effect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
- R1, R17, R2, R3, R4, R5: footprint Resistor_SMD:R_0201_0603Metric -> Resistor_SMD:R_0402_1005Metric
Connections:
- net +3V3: now also R7.1, R8.1, R9.1
- net CHIP_EN: now also C21.1, R7.2, SW1.1
- net GND: now also C21.2, C25.2, C26.2, C27.2, C28.2, D2.2 (VSS), R16.2, SW1.2, SW2.2, U4.1 (~{OE}), U4.3 (GND)
- net GPIO21_LED: now also R16.1, U4.2 (A)
- net GPIO8: now also R9.2
- net GPIO9_BOOT: now also R8.2, SW2.1
- net U0TXD_MCU: now also R14.1
- net USB_MCU_D+: now also C28.1, R13.2
- net USB_MCU_D-: now also C27.1, R12.2
- new net LED_DATA_5V: R15.1, U4.4 (Y)
- new net LED_DIN: D2.3 (DIN), R15.2
- new net U0TXD: R14.2
- new net USB_D+: R13.1
- new net USB_D-: R12.1
- new net VBUS_USB: C25.1, C26.1, D2.4 (VDD), U4.5 (VCC)
- no-connect marks 1 -> 2
Other:
- note added: "3V3 bulk and VDDA3P3 filtering"
- note added: "4 MB QSPI flash / series resistors at U1"
- note added: "40 MHz crystal / local load capacitors"
- note added: "BOOT: GPIO8 high, GPIO9 low at reset"
- note added: "EN delay and RESET"
- note added: "ESP32-C6 PICO | DIRECT-WIRED PERIPHERALS | REV A"
- note added: "GPIO headers and USB power input are on sheet 2. All GPIO signals are 3.3 V. RF values are initial values; verify matching on the assembled board."
- note added: "Native USB Serial/JTAG / connector and TVS on sheet 2"
- note added: "RF matching / 0201 unchanged"
- note removed: "01 ESP32-C6 QFN40 - external 4 MB flash"
- note removed: "02 RF chip CLCCL filter + antenna pi network"
- note removed: "03 Power decoupling - fit at the named pins"
- note removed: "04 Quad-SPI flash, powered from U1 VDD_SPI"
- note removed: "05 40 MHz crystal"
- note removed: "All GPIO signals are 3.3 V only. GPIO4/5/8/9/15 are strapping pins. Do not force strap levels during reset. GPIO21 drives the RGB LED."
- note removed: "ESP32-C6 PICO | CORE, RF & FLASH | REV A"
- note removed: "RF values are starting points only. Tune with the assembled PCB and final enclosure. 0201 RF filter; 50 ohm feed referenced to L2 GND. Keep all layers clear in antenna area."
- moved on the sheet: AE1, C10, C11, C12, C13, C14, C15, C16, C17, C18, C19, C2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

Commit message: Compact board to 20 x 29 mm and synchronize schematic fields
Move the antenna to the right with a direct feed, place the Codex logo on
the left, and retain 3.8 mm of antenna clearance. Preserve the header
pattern while trimming 0.25 mm from each side of the board.

Fix the 65 schematic field mismatches and refresh placement, BOM,
previews, dimensional checks, and layout documentation.

Validation: ERC, unconnected items, and schematic parity report zero
issues. The two pre-existing C12/C21 hole-clearance violations remain;
independent QA was skipped at the user's request.
Parts:
- AE1: AssemblyNote Pad 2 stays open with axial end copper; horizontal prototyp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 -> Pad 2 stays open with axial end copper; right-aligned horiz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
Changed lines of the file:
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@@
 			)
 		)
-		(property "AssemblyNote" "Pad 2 stays open with axial end copper; horizontal prototype, 20.5x3.5 mm all-layer clearance; RF validation required"
+		(property "AssemblyNote" "Pad 2 stays open with axial end copper; right-aligned horizontal prototype, 20x3.8 mm all-layer clearance; RF validation required"
 			(at 495.3 43.18 0)
 			(effects
